File: Projects/Mati/ESC/Design/ESC_rev01_1/MCU.kicad_sch (KiCad schematic)
At the start: 0 parts

Commit message: Update 03
STM32F4 MCU Schematic Design
Parts:
- added C1: 10u, symbol Device:C
- added C10, C9: 2.2uF, symbol Device:C
- added C11, C16, C17, C2, C3, C4, C5, C6, C7: 100n, symbol Device:C
- added C12: 1u, symbol Device:C
- added C13, C14: 10p, symbol Device:C
- added C8: 110n, symbol Device:C
- added D1, D2: LED_G, symbol Device:LED
- added D3: LED_R, symbol Device:LED
- added FB1: FerriteBead, symbol Device:FerriteBead
- added R1, R2, R3: 0R, symbol Device:R
- added R10, R8: 2k2, symbol Device:R
- added R4: 1k, symbol Device:R
- added R5, R6: 1K, symbol Device:R
- added R9: 33k, symbol Device:R
- added SW1: SW_DIP_x01, symbol Switch:SW_DIP_x01
- added TH1: 10k, symbol Device:Thermistor_NTC
- added U1: STM32F405RGTx, Package_QFP:LQFP-64_10x10mm_P0.5mm, symbol MCU_ST_STM32F4:STM32F405RGTx
- added Y1: 8M, symbol Device:Crystal
Connections:
- new net: C9.1, U1.31 (VCAP_1)
- new net: C11.1, C12.1, FB1.1, U1.13 (VDDA)
- new net: R1.2, U1.60 (BOOT0)
- new net: D1.2 (A), R4.1
- new net: D2.2 (A), R5.1
- new net: D3.2 (A), R6.1
- new net: C10.1, U1.47 (VCAP_2)
- new net: C13.1, R3.2, Y1.1
- new net: C14.1, R2.2, Y1.2
- new net +3V3: C1.1, C16.1, C2.1, C3.1, C4.1, C5.1, C6.1, C7.1, FB1.2, R1.1, R4.2, TH1.1, U1.1 (VBAT), U1.19 (VDD), U1.32 (VDD), U1.48 (VDD), U1.64 (VDD)
- new net +VDC: R9.2
- new net ADC_TEMP: R8.1, TH1.2, U1.17 (PA3)
- new net AN_IN: C17.1, R10.2, R9.1, U1.10 (PC2)
- new net BR_S01: U1.27 (PB1)
- new net BR_S02: U1.26 (PB0)
- new net CAN_RX: U1.61 (PB8)
- new net CAN_TX: U1.62 (PB9)
- new net DC_CAL: U1.33 (PB12)
- new net EN_GATE: U1.51 (PC10)
- new net FAULT: U1.53 (PC12)
- new net GND: C1.2, C10.2, C11.2, C12.2, C13.2, C14.2, C16.2, C17.2, C2.2, C3.2, C4.2, C5.2, C6.2, C7.2, C8.2, C9.2, D1.1 (K), D2.1 (K), D3.1 (K), R10.1, R8.2, SW1.1, U1.12 (VSSA), U1.18 (VSS), U1.63 (VSS)
- new net H1: U1.43 (PA10)
- new net H2: U1.42 (PA9)
- new net H3: U1.41 (PA8)
- new net HALL_1: U1.58 (PB6)
- new net HALL_2: U1.59 (PB7)
- new net HALL_3: U1.52 (PC11)
- new net L1: U1.36 (PB15)
- new net L2: U1.35 (PB14)
- new net L3: U1.34 (PB13)
- new net LED_GREEN: R5.2, U1.24 (PC4)
- new net LED_RED: R6.2, U1.25 (PC5)
- new net MISO_ADC_EXT2: U1.22 (PA6)
- new net NRST: C8.1, SW1.2, U1.7 (NRST)
- new net PH_0_P: R2.1, U1.5 (PH0)
- new net PH_1_P: R3.1, U1.6 (PH1)
- new net RX_SCL_MOSI: U1.23 (PA7), U1.29 (PB10), U1.38 (PC7)
- new net SCK_ADC_EXT: U1.21 (PA5)
- new net SENS1: U1.16 (PA2)
- new net SENS2: U1.15 (PA1)
- new net SENS3: U1.14 (PA0)
- new net SERVO: U1.57 (PB5)
- new net SWCLK: U1.49 (PA14)
- new net SWDIO: U1.46 (PA13)
- new net TEMP_MOTOR: U1.8 (PC0)
- new net TX_SDA_NSS: U1.20 (PA4), U1.30 (PB11), U1.37 (PC6)
- new net USB_DM: U1.44 (PA11)
- new net USB_DP: U1.45 (PA12)
- no-connect marks 0 -> 12
Other:
- note added: "100nF Decoupling capacitor"
- note added: "NRST internally pulled-up"
- note added: "NTC THERMISTOR"
- note added: "VOLTAGE DEVIDER"
