File: Projects/Mati/ESC/Design/ESC_rev01_1/MOSFETs.kicad_sch (KiCad schematic)
At the start: 0 parts

Commit message: Update 05
Transistors & ESC Motor Phases Schematics
Parts:
- added C39, C40: 120p, symbol Device:C
- added J4, J5, J6: Conn_01x01, symbol Connector_Generic:Conn_01x01
- added NT1, NT2, NT3, NT4, NT5, NT6, NT7, NT8: NetTie_2, symbol Device:NetTie_2
- added Q1, Q2, Q3, Q4, Q5, Q6: IRF7748L1, Package_DFN_QFN:PQFN-8-EP_6x5mm_P1.27mm_Generic, symbol Transistor_FET:IRF7748L1
- added R25, R26, R31, R32, R37, R38: 4R7, symbol Device:R
- added R27, R35, R39: 39k, symbol Device:R
- added R28, R36: 0R, symbol Device:R
- added R29, R30, R33, R34: 100R, symbol Device:R
Connections:
- new net: NT4.2, R34.2, R36.1
- new net: NT2.1, R33.2, R36.2
- new net: Q3.2 (G), R31.2
- new net: Q4.2 (G), R32.2, R35.2
- new net: Q6.2 (G), R38.2, R39.2
- new net: Q1.2 (G), R25.2
- new net: Q5.2 (G), R37.2
- new net: Q2.2 (G), R26.2, R27.2
- new net: NT3.2, R28.1, R30.2
- new net: NT1.1, R28.2, R29.2
- new net +VDC: Q1.1 (D), Q3.1 (D), Q5.1 (D)
- new net GND: NT3.1, NT4.1, NT5.1, R27.1, R35.1, R39.1
- new net H1_LOW: NT1.2, Q2.3 (S)
- new net H1_VS: NT6.2
- new net H2_LOW: NT2.2, Q4.3 (S)
- new net H2_VS: NT7.2
- new net H3_LOW: NT5.2, Q6.3 (S)
- new net H3_VS: NT8.2
- new net M_H1: R25.1
- new net M_H2: R31.1
- new net M_H3: R37.1
- new net M_L1: R26.1
- new net M_L2: R32.1
- new net M_L3: R38.1
- new net PHSAE_1: J4.1 (Pin_1), NT6.1, Q1.3 (S), Q2.1 (D)
- new net PHSAE_2: J5.1 (Pin_1), NT7.1, Q3.3 (S), Q4.1 (D)
- new net PHSAE_3: J6.1 (Pin_1), NT8.1, Q5.3 (S), Q6.1 (D)
- new net S1_N: C39.1, R29.1
- new net S1_P: C39.2, R30.1
- new net S2_N: C40.1, R33.1
- new net S2_P: C40.2, R34.1
Other:
- note added: "HX_VS"
- note added: "MCU SENSING FEEDBACK FOR EACH PASHE"
- note added: "OUTPUT_PHASE 1"
- note added: "OUTPUT_PHASE 2"
- note added: "OUTPUT_PHASE 3"
- note added: "PHASE 1"
- note added: "PHASE 2"
- note added: "PHASE 3"
- note added: "Q_CONTROL"
- note added: "Q_SOURCE"
- note added: "SENSE_1"
- note added: "SENSE_2"
