File: Projects/Mati/ESC/Design/ESC_rev01_1/CAN.kicad_sch (KiCad schematic)
At the start: 0 parts

Commit message: Update 06
USB, CAN Bus, TVS, and Schematic Completion
Parts:
- added C45, C46: 60p, symbol Device:C
- added C47: 2u2, symbol Device:C
- added D8, D9: D_TVS, symbol Device:D_TVS
- added J9: Conn_01x04, symbol Connector_Generic:Conn_01x04
- added L2: Choke_Wurth_WE-CNSW_744232090, Inductor_SMD:L_CommonMode_Wurth_WE-CNSW-1206, symbol Filter:Choke_Wurth_WE-CNSW_744232090
- added R44: 120R, symbol Device:R
- added R45, R46: 10R, symbol Device:R
- added R47: 10k, symbol Device:R
- added U3: SN65HVD230, Package_SO:SOIC-8_3.9x4.9mm_P1.27mm, symbol Interface_CAN_LIN:SN65HVD230
Connections:
- new net: C45.2, D8.2 (A2), J9.3 (Pin_3), R44.1, R45.1
- new net: R47.2, U3.8 (Rs)
- new net: C46.1, D9.1 (A1), J9.2 (Pin_2), R44.2, R46.1
- new net +3V3: C47.1, U3.3 (VCC)
- new net +5V: J9.4 (Pin_4)
- new net CAN_N: L2.3, U3.6 (CANL)
- new net CAN_P: L2.2, U3.7 (CANH)
- new net CAN_TX: U3.1 (D), U3.4 (R)
- new net GND: C45.1, C46.2, C47.2, D8.1 (A1), D9.2 (A2), J9.1 (Pin_1), R47.1, U3.2 (GND)
- new net R_CAN_N: L2.4, R46.2
- new net R_CAN_P: L2.1, R45.2
- no-connect marks 0 -> 1
Other:
- note added: "BYPASS CAPACITOR"
- note added: "CAN_H AND CAN_L TO BE ROUTED AS DIFERENTIAL PAIR"
- note added: "MODE SELECTION RESISTOR SLEW OF 15 V/uS"
- note added: "PLACE AS CLOSE AS POSSIBLE TO THE IC"
