File: Projects/Mati/ESC/Design/ESC_rev01_1/FILTERS.kicad_sch (KiCad schematic)
At the start: 0 parts

Commit message: Update 06
USB, CAN Bus, TVS, and Schematic Completion
Parts:
- added C48, C49, C50, C51, C52, C53, C55: 100n, symbol Device:C
- added C54: 4n7, symbol Device:C
- added J10: Conn_01x06, symbol Connector_Generic:Conn_01x06
- added R48, R50, R52: 2k2, symbol Device:R
- added R49, R51, R53, R54: 10k, symbol Device:R
- added R55: 0R, symbol Device:R
Connections:
- new net +3V3: C48.1, C51.1, C53.1, C55.1, R48.1, R50.1, R52.1, R54.1
- new net +5V: J10.6 (Pin_6)
- new net GND: C48.2, C49.2, C50.2, C51.2, C52.2, C53.2, C54.2, C55.2, J10.1 (Pin_1)
- new net HALL_1_IN: C49.1, J10.4 (Pin_4), R48.2, R49.1
- new net HALL_1_OUT: R49.2
- new net HALL_2_IN: C50.1, J10.3 (Pin_3), R50.2, R51.1
- new net HALL_2_OUT: R51.2
- new net HALL_3_IN: C52.1, J10.2 (Pin_2), R52.2, R53.1
- new net HALL_3_OUT: R53.2
- new net TEMP_IN: C54.1, J10.5 (Pin_5), R54.2, R55.1
- new net TEMP_MOTOR: R55.2
Other:
- note added: "HALL ENCODER OUTPUT"
- note added: "HALL_1 FILTER"
- note added: "HALL_2 FILTER"
- note added: "HALL_3 FILTER"
- note added: "TEMP_MOTOR FILTER"
- note added: "TO MCU =>"
